Commit message: Added tool_link to powerball_gripper.urdf

File: trunk/robotnik-powerball-ros-pkg/robotnik_powerball_description/urdf/powerball_gripper.urdf (robot description, URDF)
Before this commit: robot powerball, 13 links, 12 joints
Links:
- added link tool_link, mass 0.001; visual box size=0.000005 0.000005 0.000005
Joints:
- added joint gripper_base_link_tool_joint: type fixed, parent gripper_base_link, child tool_link, origin xyz=0 0 0.22 rpy=0 0 0, axis 1 0 0, limit effort=100 velocity=100
